Commit message: make changes to new mujoco

File: safety_gym/xmls/urdf/material.urdf (robot description, URDF)
Before this commit: robot cube.urdf, 1 links, 0 joints
Links:
- link baseLink: geometry collision mesh filename=material_normalized.obj scale=1 1 1; visual mesh filename=material_normalized.obj scale=1 1 1
